File: Maja V1 PCB Redesign.kicad_pcb (KiCad board)
At the start: 2 copper layers, 4 parts, among them J1 TYPE-C-31-M-12

Commit message: fixed footprint & Symbol
Parts:
- added C1: 1u, Capacitor_SMD:C_0805_2012Metric_Pad1.18x1.45mm_HandSolder, F.Cu at (-165.3, -145.9)
- added C2: 22p, Capacitor_SMD:C_0805_2012Metric_Pad1.18x1.45mm_HandSolder, F.Cu at (-120.3, -146.8)
- added C3: 0.1u, Capacitor_SMD:C_0805_2012Metric_Pad1.18x1.45mm_HandSolder, F.Cu at (-125.5, -143.5)
- added C4: 0.1u, Capacitor_SMD:C_0805_2012Metric_Pad1.18x1.45mm_HandSolder, F.Cu at (-126.2, -146.5)
- added C5: 22p, Capacitor_SMD:C_0805_2012Metric_Pad1.18x1.45mm_HandSolder, F.Cu at (-130.3, -140.5)
- added C6: 0.1u, Capacitor_SMD:C_0805_2012Metric_Pad1.18x1.45mm_HandSolder, F.Cu at (-134.0, -134.5)
- added C7: 0.1u, Capacitor_SMD:C_0805_2012Metric_Pad1.18x1.45mm_HandSolder, F.Cu at (-130.3, -137.5)
- added C8: 0.1u, Capacitor_SMD:C_0805_2012Metric_Pad1.18x1.45mm_HandSolder, F.Cu at (-120.3, -149.8)
- added D1: D, Diode_SMD:D_SOD-123, F.Cu at (21.0, -206.6)
- added D10: D, Diode_SMD:D_SOD-123, F.Cu at (26.8, -213.3)
- added D11: D, Diode_SMD:D_SOD-123, F.Cu at (32.5, -216.6)
- added D12: D, Diode_SMD:D_SOD-123, F.Cu at (128.1, -314.3)
- added D13: D, Diode_SMD:D_SOD-123, F.Cu at (21.0, -220.0)
- added D14: D, Diode_SMD:D_SOD-123, F.Cu at (110.0, -294.1)
- added D15: D, Diode_SMD:D_SOD-123, F.Cu at (60.3, -250.3)
- added D16: D, Diode_SMD:D_SOD-123, F.Cu at (26.8, -216.6)
- added D17: D, Diode_SMD:D_SOD-123, F.Cu at (-40.8, -158.1)
- added D18: D, Diode_SMD:D_SOD-123, F.Cu at (66.0, -250.3)
- added D19: D, Diode_SMD:D_SOD-123, F.Cu at (66.0, -260.4)
- added D2: D, Diode_SMD:D_SOD-123, F.Cu at (11.5, -196.4)
- added D20: D, Diode_SMD:D_SOD-123, F.Cu at (-63.8, -157.4)
- added D21: D, Diode_SMD:D_SOD-123, F.Cu at (50.8, -236.8)
- added D22: D, Diode_SMD:D_SOD-123, F.Cu at (56.5, -240.2)
- added D23: D, Diode_SMD:D_SOD-123, F.Cu at (21.0, -216.6)
- added D24: D, Diode_SMD:D_SOD-123, F.Cu at (-81.1, -157.4)
- added D25: D, Diode_SMD:D_SOD-123, F.Cu at (128.1, -317.6)
- added D26: D, Diode_SMD:D_SOD-123, F.Cu at (-98.3, -156.8)
- added D27: D, Diode_SMD:D_SOD-123, F.Cu at (11.5, -199.8)
- added D28: D, Diode_SMD:D_SOD-123, F.Cu at (133.8, -317.6)
- added D29: D, Diode_SMD:D_SOD-123, F.Cu at (-35.1, -158.1)
- added D3: D, Diode_SMD:D_SOD-123, F.Cu at (71.8, -260.4)
- added D30: D, Diode_SMD:D_SOD-123, F.Cu at (60.3, -260.4)
- added D31: D, Diode_SMD:D_SOD-123, F.Cu at (-150.1, -156.8)
- added D32: D, Diode_SMD:D_SOD-123, F.Cu at (-104.1, -156.8)
- added D33: D, Diode_SMD:D_SOD-123, F.Cu at (104.3, -300.8)
- added D34: D, Diode_SMD:D_SOD-123, F.Cu at (50.8, -240.2)
- added D35: D, Diode_SMD:D_SOD-123, F.Cu at (71.8, -253.7)
- added D36: D, Diode_SMD:D_SOD-123, F.Cu at (21.0, -209.9)
- added D37: D, Diode_SMD:D_SOD-123, F.Cu at (-132.8, -156.8)
- added D38: D, Diode_SMD:D_SOD-123, F.Cu at (-144.3, -156.8)
- added D39: D, Diode_SMD:D_SOD-123, F.Cu at (21.0, -203.2)
- added D4: D, Diode_SMD:D_SOD-123, F.Cu at (104.3, -297.4)
- added D40: D, Diode_SMD:D_SOD-123, F.Cu at (-23.6, -158.1)
- added D41: D, Diode_SMD:D_SOD-123, F.Cu at (-109.8, -156.8)
- added D42: D, Diode_SMD:D_SOD-123, F.Cu at (26.8, -220.0)
- added D43: D, Diode_SMD:D_SOD-123, F.Cu at (110.0, -300.8)
- added D44: D, Diode_SMD:D_SOD-123, F.Cu at (60.3, -253.7)
- added D45: D, Diode_SMD:D_SOD-123, F.Cu at (-52.3, -157.4)
- added D46: D, Diode_SMD:D_SOD-123, F.Cu at (-86.8, -157.4)
- added D47: D, Diode_SMD:D_SOD-123, F.Cu at (21.0, -213.3)
- added D48: D, Diode_SMD:D_SOD-123, F.Cu at (-127.1, -156.8)
- added D49: D, Diode_SMD:D_SOD-123, F.Cu at (60.3, -257.0)
- added D5: D, Diode_SMD:D_SOD-123, F.Cu at (60.3, -247.0)
- added D50: D, Diode_SMD:D_SOD-123, F.Cu at (115.8, -300.8)
- added D51: D, Diode_SMD:D_SOD-123, F.Cu at (-29.3, -158.1)
- added D52: D, Diode_SMD:D_SOD-123, F.Cu at (104.3, -294.1)
- added D53: D, Diode_SMD:D_SOD-123, F.Cu at (104.3, -290.7)
- added D54: D, Diode_SMD:D_SOD-123, F.Cu at (94.8, -280.6)
- added D55: D, Diode_SMD:D_SOD-123, F.Cu at (66.0, -253.7)
- added D56: D, Diode_SMD:D_SOD-123, F.Cu at (128.1, -321.0)
- added D57: D, Diode_SMD:D_SOD-123, F.Cu at (-115.6, -156.8)
- added D58: D, Diode_SMD:D_SOD-123, F.Cu at (-69.6, -157.4)
- added D59: D, Diode_SMD:D_SOD-123, F.Cu at (-92.6, -156.8)
- added D6: D, Diode_SMD:D_SOD-123, F.Cu at (-121.3, -156.8)
- added D60: D, Diode_SMD:D_SOD-123, F.Cu at (32.5, -220.0)
- added D61: D, Diode_SMD:D_SOD-123, F.Cu at (-75.3, -157.4)
- added D62: D, Diode_SMD:D_SOD-123, F.Cu at (-46.6, -158.1)
- added D63: D, Diode_SMD:D_SOD-123, F.Cu at (-58.1, -157.4)
- added D64: D, Diode_SMD:D_SOD-123, F.Cu at (110.0, -297.4)
- added D65: D, Diode_SMD:D_SOD-123, F.Cu at (94.8, -277.2)
- added D66: D, Diode_SMD:D_SOD-123, F.Cu at (-8.69, -175.6)
- added D67: D, Diode_SMD:D_SOD-123, F.Cu at (66.0, -257.0)
- added D68: D, Diode_SMD:D_SOD-123, F.Cu at (133.8, -321.0)
- added D7: D, Diode_SMD:D_SOD-123, F.Cu at (71.8, -257.0)
- added D8: D, Diode_SMD:D_SOD-123, F.Cu at (-8.69, -178.9)
- added D9: D, Diode_SMD:D_SOD-123, F.Cu at (-138.6, -156.8)
- added F1: 500m, Fuse:Fuse_1206_3216Metric_Pad1.42x1.75mm_HandSolder, F.Cu at (-125.7, -149.7)
- added J2: AVR-ISP-6, random-keyboard-parts:Reset_Pretty, F.Cu at (-139.5, -132.4)
- added K1: esc, Keyboard Component:SW_Cherry_MX_1.00u_PCB, F.Cu at (-68.6, -141.6)
- added K10: 9, Keyboard Component:SW_Cherry_MX_1.00u_PCB, F.Cu at (-80.9, -234.9)
- added K11: 0, Keyboard Component:SW_Cherry_MX_1.00u_PCB, F.Cu at (-79.7, -174.3)
- added K12: -, Keyboard Component:SW_Cherry_MX_1.00u_PCB, F.Cu at (-59.5, -194.5)
- added K13: =, Keyboard Component:SW_Cherry_MX_1.00u_PCB, F.Cu at (64.1, -277.2)
- added K14: ~, Keyboard Component:SW_Cherry_MX_1.00u_PCB, F.Cu at (9.44, -257.0)
- added K15: split backspace, Keyboard Component:SW_Cherry_MX_1.00u_PCB, F.Cu at (10.6, -216.6)
- added K16: macro1, Keyboard Component:SW_Cherry_MX_1.00u_PCB, F.Cu at (-7.15, -297.4)
- added K17: tab, Keyboard Component:SW_Cherry_MX_1.50u_PCB, F.Cu at (-67.6, -122.6)
- added K18: q, Keyboard Component:SW_Cherry_MX_1.00u_PCB, F.Cu at (-43.8, -122.6)
- added K19: w, Keyboard Component:SW_Cherry_MX_1.00u_PCB, F.Cu at (-42.1, -103.5)
- added K2: 1, Keyboard Component:SW_Cherry_MX_1.00u_PCB, F.Cu at (-49.5, -141.6)
- added K20: e, Keyboard Component:SW_Cherry_MX_1.00u_PCB, F.Cu at (-9.61, -216.0)
- added K21: r, Keyboard Component:SW_Cherry_MX_1.00u_PCB, F.Cu at (-70.2, -214.7)
- added K22: t, Keyboard Component:SW_Cherry_MX_1.00u_PCB, F.Cu at (-50.0, -215.3)
- added K23: y, Keyboard Component:SW_Cherry_MX_1.00u_PCB, F.Cu at (117.7, -317.6)
- added K24: u, Keyboard Component:SW_Cherry_MX_1.00u_PCB, F.Cu at (-39.3, -195.1)
- added K25: i, Keyboard Component:SW_Cherry_MX_1.00u_PCB, F.Cu at (29.6, -257.0)
- added K26: o, Keyboard Component:SW_Cherry_MX_1.00u_PCB, F.Cu at (-51.2, -255.7)
- added K27: p, Keyboard Component:SW_Cherry_MX_1.00u_PCB, F.Cu at (97.5, -317.6)
- added K28: [, Keyboard Component:SW_Cherry_MX_1.00u_PCB, F.Cu at (-10.8, -257.0)
- added K29: ], Keyboard Component:SW_Cherry_MX_1.00u_PCB, F.Cu at (-140.3, -173.7)
- added K3: 2, Keyboard Component:SW_Cherry_MX_1.00u_PCB, F.Cu at (-30.5, -143.2)
- added K30: \, Keyboard Component:SW_Cherry_MX_1.50u_PCB, F.Cu at (-135.6, -214.1)
- added K31: macro 2, Keyboard Component:SW_Cherry_MX_1.00u_PCB, F.Cu at (36.9, -317.6)
- added K32: Caps, Keyboard Component:SW_Cherry_MX_1.75u_PCB, F.Cu at (-68.3, -103.5)
- added K33: a, Keyboard Component:SW_Cherry_MX_1.00u_PCB, F.Cu at (-90.4, -214.7)
- added K34: s, Keyboard Component:SW_Cherry_MX_1.00u_PCB, F.Cu at (-99.9, -173.7)
- added K35: d, Keyboard Component:SW_Cherry_MX_1.00u_PCB, F.Cu at (57.1, -317.6)
- added K36: f, Keyboard Component:SW_Cherry_MX_1.00u_PCB, F.Cu at (-71.4, -255.7)
- added K37: g, Keyboard Component:SW_Cherry_MX_1.00u_PCB, F.Cu at (-40.5, -235.5)
- added K38: h, Keyboard Component:SW_Cherry_MX_1.00u_PCB, F.Cu at (40.3, -236.8)
- added K39: j, Keyboard Component:SW_Cherry_MX_1.00u_PCB, F.Cu at (20.1, -236.8)
- added K4: 3, Keyboard Component:SW_Cherry_MX_1.00u_PCB, F.Cu at (27.8, -181.8)
- added K40: k, Keyboard Component:SW_Cherry_MX_1.00u_PCB, F.Cu at (53.5, -297.4)
- added K41: l, Keyboard Component:SW_Cherry_MX_1.00u_PCB, F.Cu at (73.7, -297.4)
- added K42: ;, Keyboard Component:SW_Cherry_MX_1.00u_PCB, F.Cu at (49.8, -257.0)
- added K43: ', Keyboard Component:SW_Cherry_MX_1.00u_PCB, F.Cu at (-36.9, -276.6)
- added K44: enter, Keyboard Component:SW_Cherry_MX_2.25u_PCB, F.Cu at (-128.4, -275.9)
- added K45: macro 3, Keyboard Component:SW_Cherry_MX_1.00u_PCB, F.Cu at (-39.3, -174.9)
- added K46: shift, Keyboard Component:SW_Cherry_MX_2.25u_PCB, F.Cu at (-74.9, -317.6)
- added K47: z, Keyboard Component:SW_Cherry_MX_1.00u_PCB, F.Cu at (77.3, -317.6)
- added K48: x, Keyboard Component:SW_Cherry_MX_1.00u_PCB, F.Cu at (-120.1, -173.7)
- added K49: c, Keyboard Component:SW_Cherry_MX_1.00u_PCB, F.Cu at (-27.3, -297.4)
- added K5: 4, Keyboard Component:SW_Cherry_MX_1.00u_PCB, F.Cu at (23.7, -277.2)
- added K50: v, Keyboard Component:SW_Cherry_MX_1.00u_PCB, F.Cu at (-20.3, -236.2)
- added K51: b, Keyboard Component:SW_Cherry_MX_1.00u_PCB, F.Cu at (3.52, -277.2)
- added K52: fn, Keyboard Component:SW_Cherry_MX_1.00u_PCB, F.Cu at (92.2, -179.7)
- added K53: n, Keyboard Component:SW_Cherry_MX_1.00u_PCB, F.Cu at (33.3, -297.4)
- added K54: m, Keyboard Component:SW_Cherry_MX_1.00u_PCB, F.Cu at (16.7, -317.6)
- added K55: ,, Keyboard Component:SW_Cherry_MX_1.00u_PCB, F.Cu at (-31.0, -256.4)
- added K56: ., Keyboard Component:SW_Cherry_MX_1.00u_PCB, F.Cu at (13.1, -297.4)
- added K57: /, Keyboard Component:SW_Cherry_MX_1.00u_PCB, F.Cu at (84.3, -277.2)
- added K58: shift right, Keyboard Component:SW_Cherry_MX_1.75u_PCB, F.Cu at (-133.2, -234.3)
- added K59: up, Keyboard Component:SW_Cherry_MX_1.00u_PCB, F.Cu at (2.88, -163.9)
- added K6: 5, Keyboard Component:SW_Cherry_MX_1.00u_PCB, F.Cu at (-120.1, -193.9)
- added K60: ctrl left, Keyboard Component:SW_Cherry_MX_1.50u_PCB, F.Cu at (-61.8, -275.9)
- added K61: alt right, Keyboard Component:SW_Cherry_MX_1.50u_PCB, F.Cu at (-96.3, -255.1)
- added K62: space left, Keyboard Component:SW_Cherry_MX_2.25u_PCB, F.Cu at (-128.4, -296.8)
- added K63: code, Keyboard Component:SW_Cherry_MX_1.00u_PCB, F.Cu at (-101.1, -234.9)
- added K64: space right, Keyboard Component:SW_Cherry_MX_2.75u_PCB, F.Cu at (-123.2, -317.6)
- added K65: ctrl right, Keyboard Component:SW_Cherry_MX_1.50u_PCB, F.Cu at (-91.6, -275.9)
- added K66: left, Keyboard Component:SW_Cherry_MX_1.00u_PCB, F.Cu at (43.9, -277.2)
- added K67: down, Keyboard Component:SW_Cherry_MX_1.00u_PCB, F.Cu at (-60.7, -235.5)
- added K68: right, Keyboard Component:SW_Cherry_MX_1.00u_PCB, F.Cu at (-140.3, -193.9)
- added K69: backspace, Keyboard Component:SW_Cherry_MX_2.00u_PCB, F.Cu at (-130.8, -255.1)
- added K7: 6, Keyboard Component:SW_Cherry_MX_1.00u_PCB, F.Cu at (-16.7, -277.2)
- added K70: space left 2, Keyboard Component:SW_Cherry_MX_2.00u_PCB, F.Cu at (-86.8, -296.8)
- added K71: code 2, Keyboard Component:SW_Cherry_MX_1.25u_PCB, F.Cu at (-5.92, -317.6)
- added K72: Caps steped, Keyboard Component:SW_Cherry_MX_1.75u_PCB, F.Cu at (-73.0, -103.5)
- added K8: 7, Keyboard Component:SW_Cherry_MX_1.00u_PCB, F.Cu at (93.9, -297.4)
- added K9: 8, Keyboard Component:SW_Cherry_MX_1.00u_PCB, F.Cu at (-99.9, -193.9)
- added R1: 5.1k, Resistor_SMD:R_0805_2012Metric_Pad1.20x1.40mm_HandSolder, F.Cu at (-125.5, -140.6)
- added R2: 5.1k, Resistor_SMD:R_0805_2012Metric_Pad1.20x1.40mm_HandSolder, F.Cu at (-125.5, -137.6)
- added R3: 10k, Resistor_SMD:R_0805_2012Metric_Pad1.20x1.40mm_HandSolder, F.Cu at (-129.2, -134.6)
- added R4: 22, Resistor_SMD:R_0805_2012Metric_Pad1.20x1.40mm_HandSolder, F.Cu at (-125.0, -127.1)
- added R5: 22, Resistor_SMD:R_0805_2012Metric_Pad1.20x1.40mm_HandSolder, F.Cu at (-120.7, -143.8)
- added R6: 10k, Resistor_SMD:R_0805_2012Metric_Pad1.20x1.40mm_HandSolder, F.Cu at (-115.5, -149.9)
- added REF**: SW_Cherry_MX_2.75u_PCB, Button_Switch_Keyboard:SW_Cherry_MX_2.75u_PCB, F.Cu at (-96.5, 20.0)
- added S1: SKQGAFE010, Keyboard Component:SW_SKQGAFE010, F.Cu at (-158.9, -128.7)
- added U1: ATmega32U4-M, Package_DFN_QFN:QFN-44-1EP_7x7mm_P0.5mm_EP5.2x5.2mm, F.Cu at (-143.5, -145.9)
- added U2: PRTR5V0U2X, random-keyboard-parts:SOT143B, F.Cu at (-115.8, -146.4)
- added Y1: Crystal_GND24_Small, Crystal:Crystal_SMD_3225-4Pin_3.2x2.5mm, F.Cu at (-135.3, -139.8)
- moved J1 247.3 mm to (-155.6, 73.8)
- moved REF** 217.7 mm to (-149.9, 42.9)
- moved REF** 217.7 mm to (-139.7, 60.6)
- moved REF** 217.7 mm to (-139.7, 50.5)
Connections:
- J1 pad A1B12: unconnected-(J1-PadA1B12) -> GND
- J1 pad A4B9: unconnected-(J1-PadA4B9) -> VCC
- J1 pad A5: unconnected-(J1-PadA5) -> Net-(J1-PadA5)
- J1 pad A6: unconnected-(J1-PadA6) -> Net-(J1-PadA6)
- J1 pad A7: unconnected-(J1-PadA7) -> Net-(J1-PadA7)
- J1 pad B1A12: unconnected-(J1-PadB1A12) -> GND
- J1 pad B4A9: unconnected-(J1-PadB4A9) -> VCC
- J1 pad B5: unconnected-(J1-PadB5) -> Net-(J1-PadB5)
- J1 pad B6: unconnected-(J1-PadB6) -> Net-(J1-PadA6)
- J1 pad B7: unconnected-(J1-PadB7) -> Net-(J1-PadA7)
- J1 pad S1: Net-(J1-PadS1) -> GND
- J1 pad S2: Net-(J1-PadS1) -> GND
- J1 pad S3: Net-(J1-PadS1) -> GND
- J1 pad S4: Net-(J1-PadS1) -> GND
Other:
- board outline added: 345.1 x 138.7 mm

Commit message: key placement
Parts:
- added REF**: QFP80P1200X1200X120-44N, Keyboard Component:QFP80P1200X1200X120-44N, B.Cu at (52.4, -93.2)
- C1, C2, C3, C4, C5, C6, C7, C8, D1, D10, D11, D12, D13, D14, D15, D16, D17, D18, D19, D2, D20, D21, D22, D23, D24, D25, D26, D27, D28, D29, D3, D30, D31, D32, D33, D34, D35, D36, D37, D38, D39, D4, D40, D41, D42, D43, D44, D45, D46, D47, D48, D49, D5, D50, D51, D52, D53, D54, D55, D56, D57, D58, D59, D6, D60, D61, D62, D63, D64, D65, D66, D67, D68, D7, D8, D9, F1, J2, R1, R2, R3, R4, R5, R6, S1, U1, U2, Y1: moved to B.Cu
- moved K68 407.8 mm to (244.6, -59.3)
- moved K44 376.1 mm to (205.1, -102.2)
- moved K58 360.6 mm to (194.2, -83.2)
- moved K30 356.8 mm to (209.0, -121.3)
- moved K69 350.7 mm to (200.6, -140.3)
- moved K64 337.8 mm to (90.8, -56.3), turned to 10 degrees
- moved K67 336.1 mm to (225.6, -59.3)
- moved K29 329.7 mm to (185.2, -121.3)
- moved J1 327.4 mm to (79.8, -153.7), turned to 180 degrees
- moved K65 308.8 mm to (131.0, -61.8), turned to 10 degrees
- moved K16 296.8 mm to (244.6, -140.3)
- moved K45 293.1 mm to (244.6, -102.2)
- moved K31 285.9 mm to (244.6, -121.3)
- moved K62 281.0 mm to (17.4, -56.6), turned to -10 degrees
- moved K43 273.7 mm to (174.1, -102.2)
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