File: Maja V1 PCB Redesign.kicad_pcb (KiCad board)
At the start: 2 copper layers, 345.1 x 138.7 mm, 166 parts, among them J1 TYPE-C-31-M-12, J2 AVR-ISP-6, K1 esc, K10 9, K11 0, K12 -, K13 =, K15 split backspace, K16 macro1, K17 tab, K18 q, K19 w, K2 1, K20 e, K21 r, K22 t, K23 y, K24 u, K25 i, K26 o, K27 p, K28 [, K29 ], K3 2, K30 \, K31 macro 2, K32 Caps, K33 a, K34 s, K35 d, K36 f, K37 g, K38 h, K39 j, K4 3, K40 k, K41 l, K42 ;, K43 ', K44 enter, K45 macro 3, K46 shift, K47 z, K48 x, K49 c, K5 4, K50 v, K51 b, K52 fn, K53 n, K54 m, K55 ,, K56 ., K57 /, K58 shift right, K59 up, K6 5, K60 ctrl left, K61 alt right, K62 space left, K63 code, K64 space right, K65 ctrl right, K66 left, K67 down, K68 right, K69 backspace, K7 6, K70 space left 2, K71 code 2, K72 Caps steped, K8 7, K9 8, U1 ATmega32U4-M, U2 PRTR5V0U2X, Y1 Crystal_GND24_Small

Commit message: MCU
Parts:
- added J3: Connector_Generic_Conn_01x04, Connector_JST:JST_SH_SM04B-SRSS-TB_1x04-1MP_P1.00mm_Horizontal, B.Cu at (57.1, -138.2)
- moved R5 134.5 mm to (53.1, -99.4), turned to -90 degrees
- moved R4 117.0 mm to (51.0, -99.4), turned to -90 degrees
- moved U2 114.9 mm to (61.6, -125.5)
- moved F1 106.5 mm to (79.9, -141.2), turned to 0 degrees
- moved R2 97.6 mm to (88.5, -144.3), turned to 0 degrees
- moved R1 92.0 mm to (70.3, -143.8)
- moved REF** 3.33 mm to (55.4, -85.8)
- moved U1 3.33 mm to (55.4, -85.8)
Connections:
- REF** pad 10: (no net) -> MOSI
- REF** pad 11: (no net) -> MISO
- REF** pad 12: (no net) -> ROW 2
- REF** pad 13: (no net) -> RESET
- REF** pad 14: (no net) -> +5V
- REF** pad 15: (no net) -> GND
- REF** pad 16: (no net) -> XTAL2
- REF** pad 17: (no net) -> XTAL1
- REF** pad 18: (no net) -> COL7
- REF** pad 19: (no net) -> COL8
- REF** pad 2: (no net) -> +5V
- REF** pad 20: (no net) -> COL9
- REF** pad 21: (no net) -> COL10
- REF** pad 22: (no net) -> COL11
- REF** pad 23: (no net) -> GND
- REF** pad 24: (no net) -> +5V
- REF** pad 25: (no net) -> COL12
- REF** pad 26: (no net) -> COL13
- REF** pad 27: (no net) -> COL14
- REF** pad 28: (no net) -> COL15
- REF** pad 29: (no net) -> ROW3
- REF** pad 3: (no net) -> D-
- REF** pad 30: (no net) -> ROW4
- REF** pad 32: (no net) -> COL6
- REF** pad 33: (no net) -> Net-(R6-Pad1)
- REF** pad 34: (no net) -> +5V
- REF** pad 35: (no net) -> GND
- REF** pad 36: (no net) -> COL5
- REF** pad 37: (no net) -> COL4
- REF** pad 38: (no net) -> COL3
- REF** pad 39: (no net) -> COL2
- REF** pad 4: (no net) -> D+
- REF** pad 40: (no net) -> COL1
- REF** pad 41: (no net) -> COL0
- REF** pad 43: (no net) -> GND
- REF** pad 44: (no net) -> +5V
- REF** pad 5: (no net) -> GND
- REF** pad 6: (no net) -> Net-(C1-Pad1)
- REF** pad 7: (no net) -> +5V
- REF** pad 8: (no net) -> ROW1
- REF** pad 9: (no net) -> SCK
- U1 pad 18: COL0 -> COL7
- U1 pad 19: COL1 -> COL8
- U1 pad 20: COL2 -> COL9
- U1 pad 21: COL3 -> COL10
- U1 pad 22: COL5 -> COL11
- U1 pad 25: COL4 -> COL12
- U1 pad 26: COL6 -> COL13
- U1 pad 27: unconnected-(U1-Pad27) -> COL14
- U1 pad 28: ROW4 -> COL15
- U1 pad 30: COL13 -> ROW4
- U1 pad 31: COL15 -> unconnected-(U1-Pad31)
- U1 pad 32: COL14 -> COL6
- U1 pad 36: COL12 -> COL5
- U1 pad 37: COL11 -> COL4
- U1 pad 38: COL10 -> COL3
- U1 pad 39: COL9 -> COL2
- U1 pad 40: COL8 -> COL1
- U1 pad 41: COL7 -> COL0
Routing:
- net +5V: track 0.00 -> 18.6 mm
- net GND: track 0.00 -> 15.5 mm
- net MISO: track 0.00 -> 3.48 mm
- net ROW0: track 0.00 -> 3.48 mm
- net COL11: track 0.00 -> 3.47 mm
- net Net-(R6-Pad1): track 0.00 -> 3.38 mm
- net ROW 2: track 0.00 -> 3.38 mm
- net MOSI: track 0.00 -> 3.26 mm
- net COL10: track 0.00 -> 3.25 mm
- net COL6: track 0.00 -> 3.06 mm
- net RESET: track 0.00 -> 3.06 mm
- net COL9: track 0.00 -> 2.94 mm
- net COL5: track 0.00 -> 2.94 mm
- net SCK: track 0.00 -> 2.94 mm
- net D-: track 0.00 -> 2.94 mm
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
Commit message: tracing 1
Parts:
- C3, C4, C6, C7: value 0.1u -> 100nF
- C8: value 0.1u -> 10uF
- J1: moved to B.Cu
- moved R6 163.3 mm to (45.5, -75.9)
- moved C4 162.4 mm to (56.6, -73.5), turned to 0 degrees
- moved C2 158.6 mm to (68.5, -81.2), turned to 0 degrees
- moved C8 151.4 mm to (43.1, -87.0), turned to -90 degrees
- moved C3 148.1 mm to (63.0, -86.2), turned to -90 degrees
- moved C5 148.0 mm to (68.5, -83.4), turned to 0 degrees
- moved Y1 146.8 mm to (63.8, -82.3), turned to 90 degrees
- moved C7 146.3 mm to (43.1, -79.3), turned to 90 degrees
- moved C1 141.1 mm to (52.9, -94.4)
- moved C6 130.8 mm to (47.9, -91.8)
- moved R3 5.37 mm to (36.8, -217.4)
- moved REF** 4.16 mm to (52.6, -82.7)
- moved U1 4.16 mm to (52.6, -82.7)
- moved D38 0.88 mm to (82.8, -91.0)
- moved D37 0.77 mm to (40.0, -90.2)
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Routing:
- net COL0: track 2.81 -> 85.9 mm
- net COL1: track 2.69 -> 77.0 mm

Commit message: routing 1
Routing:
- net (no net): track 0.00 -> 807.4 mm
- net COL4: track 2.84 -> 103.5 mm
- net COL3: track 2.69 -> 99.5 mm
- net COL0: track 85.9 -> 2.81 mm
- net COL5: track 2.94 -> 67.6 mm
- net COL2: track 2.56 -> 60.3 mm
- net COL1: track 77.0 -> 85.3 mm
Other:
- outline, holes or cut-outs redrawn

Commit message: routing 2
Routing:
- net COL4: track 103.5 -> 272.6 mm
- net COL13: track 2.81 -> 135.1 mm
- net COL10: track 3.25 -> 131.0 mm
- net COL14: track 2.69 -> 124.4 mm
- net COL6: track 3.06 -> 91.9 mm
- net COL11: track 3.47 -> 91.2 mm
- net COL15: track 2.56 -> 85.6 mm
- net COL5: track 67.6 -> 114.5 mm
- net COL3: track 99.5 -> 146.3 mm
- net COL2: track 60.3 -> 105.4 mm
- net COL1: track 85.3 -> 91.5 mm

Commit message: finish col routing
Routing:
- net COL10: track 131.0 -> 299.4 mm
- net COL8: track 2.81 -> 163.1 mm
- net COL9: track 2.94 -> 150.9 mm
- net COL0: track 2.81 -> 135.1 mm
- net COL12: track 2.94 -> 104.4 mm
- net COL7: track 2.69 -> 94.6 mm
- net COL14: track 124.4 -> 181.8 mm
- net COL11: track 91.2 -> 146.3 mm
- net COL13: track 135.1 -> 167.0 mm
- net ROW0: track 3.48 -> 12.2 mm
- net Net-(D1-Pad2): track 0.00 -> 4.70 mm

Commit message: test silkscreen
Parts:
- added ?: , , F.Cu at (230.0, 183.5)
- added ?: , , F.Cu at (460.4, 192.9)
- moved D44 268.0 mm to (342.7, 132.4)
- moved D54 268.0 mm to (246.5, 154.9)
- moved D65 268.0 mm to (268.9, 172.0)
- moved D9 268.0 mm to (231.9, 99.5)
- moved K37 268.0 mm to (168.3, 140.8)
- moved K41 268.0 mm to (266.1, 130.4)
- moved R1 268.0 mm to (202.9, 89.1)
- moved R4 268.0 mm to (183.6, 133.5)
- moved C1 268.0 mm to (185.5, 138.5)
- moved C2 268.0 mm to (201.1, 151.7)
- moved C3 268.0 mm to (195.6, 146.7)
- moved C4 268.0 mm to (189.2, 159.4)
- moved C5 268.0 mm to (201.1, 149.5)
- moved C6 268.0 mm to (180.5, 141.1)
- moved C7 268.0 mm to (175.7, 153.6)
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
Commit message: routing
Parts:
- removed ? (x2): , 
- moved D64 24.9 mm to (205.1, 185.2)
- moved D16 17.5 mm to (366.2, 101.1)
- moved D31 17.5 mm to (366.2, 120.1)
- moved D45 17.4 mm to (366.2, 139.1)
- moved D65 17.2 mm to (253.5, 179.7)
- moved D51 16.9 mm to (162.5, 167.2)
- moved D68 16.8 mm to (366.8, 181.7)
- moved D37 16.1 mm to (156.8, 145.9)
- moved D44 9.98 mm to (351.3, 137.5)
- moved D48 6.69 mm to (122.2, 160.6)
- moved D1 6.61 mm to (69.3, 99.5)
- moved D4 6.61 mm to (127.3, 103.5)
- moved D2 6.61 mm to (88.4, 99.5)
- moved D3 6.58 mm to (107.4, 97.9)
- moved D59 6.57 mm to (363.6, 162.7)
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Routing:
- net (no net): track 807.4 -> 3554.8 mm
- net ROW4: track 2.81 -> 296.0 mm
- net ROW0: track 12.2 -> 281.4 mm
- net ROW1: track 2.81 -> 269.2 mm
- net ROW3: track 2.69 -> 257.9 mm
- net ROW 2: track 3.38 -> 245.9 mm
- net Net-(D62-Pad2): track 0.00 -> 21.7 mm
- net Net-(D51-Pad2): track 0.00 -> 19.0 mm
- net Net-(D37-Pad2): track 0.00 -> 17.0 mm
- net Net-(D32-Pad2): track 0.00 -> 16.3 mm
- net Net-(D49-Pad2): track 0.00 -> 12.4 mm
- net Net-(D6-Pad2): track 0.00 -> 12.2 mm
- net Net-(D48-Pad2): track 0.00 -> 12.0 mm
- net Net-(D5-Pad2): track 0.00 -> 12.0 mm
- net Net-(D47-Pad2): track 0.00 -> 12.0 mm
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
Commit message: routing
Routing:
- net COL0: track 135.1 -> 261.3 mm
- net COL1: track 91.8 -> 200.1 mm, vias 0 -> 1
- net COL2: track 105.4 -> 184.8 mm, vias 0 -> 1
- net COL3: track 146.3 -> 204.2 mm, vias 0 -> 1
- net COL6: track 91.9 -> 130.6 mm
- net Net-(D14-Pad2): track 0.00 -> 26.6 mm
- net Net-(D64-Pad2): track 0.00 -> 21.5 mm
- net Net-(D16-Pad2): track 0.00 -> 19.2 mm
- net COL5: track 114.5 -> 133.3 mm, vias 0 -> 1
- net Net-(D31-Pad2): track 0.00 -> 17.9 mm
- net Net-(D45-Pad2): track 0.00 -> 17.7 mm
- net Net-(D65-Pad2): track 0.00 -> 17.3 mm
- net Net-(D68-Pad2): track 0.00 -> 17.1 mm
- net Net-(D44-Pad2): track 0.00 -> 15.7 mm
- net Net-(D67-Pad2): track 0.00 -> 12.1 mm
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