File: Maja V1 PCB Redesign.kicad_pcb (KiCad board)
At the start: 2 copper layers, 345.1 x 138.7 mm, 167 parts, among them J1 TYPE-C-31-M-12, J2 AVR-ISP-6, J3 Connector_Generic_Conn_01x04, K1 esc, K10 9, K11 0, K12 -, K13 =, K15 split backspace, K16 macro1, K17 tab, K18 q, K19 w, K2 1, K20 e, K21 r, K22 t, K23 y, K24 u, K25 i, K26 o, K27 p, K28 [, K29 ], K3 2, K30 \, K31 macro 2, K32 Caps, K33 a, K34 s, K35 d, K36 f, K37 g, K38 h, K39 j, K4 3, K40 k, K41 l, K42 ;, K43 ', K44 enter, K45 macro 3, K46 shift, K47 z, K48 x, K49 c, K5 4, K50 v, K51 b, K52 fn, K53 n, K54 m, K55 ,, K56 ., K57 /, K58 shift right, K59 up, K6 5, K60 ctrl left, K61 alt right, K62 space left, K63 code, K64 space right, K65 ctrl right, K66 left, K67 down, K68 right, K69 backspace, K7 6, K70 space left 2, K71 code 2, K72 Caps steped, K8 7, K9 8, U1 ATmega32U4-M, U2 PRTR5V0U2X, Y1 Crystal_GND24_Small

Commit message: routing
Parts:
- moved D36 16.2 mm to (137.7, 142.8)
- moved D37 15.9 mm to (172.3, 149.5)
- moved C2 14.6 mm to (199.8, 137.2)
- moved C3 14.6 mm to (194.2, 132.2)
- moved Y1 14.6 mm to (195.0, 136.1)
- moved C6 14.6 mm to (179.2, 126.6)
- moved R5 14.6 mm to (184.3, 119.0)
- moved C1 14.6 mm to (184.1, 124.0)
- moved C4 14.6 mm to (187.9, 144.9)
- moved C5 14.6 mm to (199.8, 135.0)
- moved C8 14.6 mm to (174.4, 131.4)
- moved R4 14.6 mm to (182.3, 119.0)
- moved R6 14.6 mm to (176.8, 142.5)
- moved REF** 14.6 mm to (183.9, 135.7)
- moved U1 14.6 mm to (183.9, 135.7)
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Connections:
- REF** pad 29: ROW3 -> ROW4
- REF** pad 30: ROW4 -> ROW3
- U1 pad 29: ROW3 -> ROW4
- U1 pad 30: ROW4 -> ROW3
Routing:
- net COL15: track 85.6 -> 268.6 mm, vias 0 -> 1
- net COL4: track 272.6 -> 337.8 mm, vias 0 -> 1
- net ROW4: track 296.0 -> 331.7 mm
- net ROW3: track 257.9 -> 292.1 mm
- net COL5: track 133.3 -> 160.3 mm
- net COL3: track 204.2 -> 230.2 mm
- net COL2: track 184.8 -> 210.5 mm
- net COL1: track 200.1 -> 222.8 mm
- net COL6: track 130.6 -> 148.7 mm
- net ROW 2: track 246.4 -> 264.0 mm, vias 0 -> 2
- net COL0: track 261.3 -> 276.3 mm
- net Net-(D36-Pad2): track 10.6 -> 0.00 mm
- net Net-(D63-Pad2): track 2.52 -> 11.9 mm
- net Net-(D37-Pad2): track 17.0 -> 13.2 mm
Other:
- board size 345.1 x 138.7 mm -> 345.1 x 120.7 mm

Commit message: routing
Parts:
- moved C4 1.48 mm to (189.3, 144.5)
- moved C3 1.06 mm to (195.0, 132.9), turned to 180 degrees
Connections:
- REF** pad 18: COL7 -> COL15
- REF** pad 19: COL8 -> COL14
- REF** pad 20: COL9 -> COL13
- REF** pad 21: COL10 -> COL12
- REF** pad 25: COL12 -> COL10
- REF** pad 26: COL13 -> COL9
- REF** pad 27: COL14 -> COL8
- REF** pad 28: COL15 -> COL7
- U1 pad 18: COL7 -> COL15
- U1 pad 19: COL8 -> COL14
- U1 pad 20: COL9 -> COL13
- U1 pad 21: COL10 -> COL12
- U1 pad 25: COL12 -> COL10
- U1 pad 26: COL13 -> COL9
- U1 pad 27: COL14 -> COL8
- U1 pad 28: COL15 -> COL7
Routing:
- net COL14: track 181.8 -> 357.1 mm, vias 0 -> 1
- net (no net): track 3554.8 -> 3404.4 mm
- net COL13: track 167.0 -> 301.0 mm, vias 0 -> 1
- net COL12: track 104.4 -> 216.6 mm, vias 0 -> 2
- net COL11: track 146.3 -> 237.7 mm, vias 0 -> 3
- net COL10: track 299.4 -> 370.8 mm, vias 0 -> 5
- net COL9: track 150.9 -> 207.9 mm, vias 0 -> 3
- net COL8: track 163.1 -> 199.4 mm, vias 0 -> 5
- net COL7: track 94.6 -> 116.2 mm, vias 0 -> 3
- net Net-(D36-Pad2): track 0.00 -> 16.2 mm
- net ROW4: track 331.7 -> 347.8 mm
- net COL15: track 268.6 -> 280.5 mm
- net ROW3: track 292.1 -> 301.1 mm
- net COL6: track 148.7 -> 157.1 mm, vias 0 -> 4
- net COL4: track 337.8 -> 334.7 mm, vias 1 -> 5
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
Commit message: routing
Parts:
- moved J2 128.7 mm to (229.9, 131.7), turned to 90 degrees
- moved R3 126.7 mm to (210.4, 135.3), turned to 100 degrees
- moved S1 119.1 mm to (217.3, 134.1), turned to -170 degrees
- moved U2 23.4 mm to (212.4, 92.7)
- moved R1 13.6 mm to (216.4, 89.4), turned to 0 degrees
- moved R2 12.7 mm to (208.5, 89.4), turned to 180 degrees
- moved F1 6.53 mm to (206.9, 95.0), turned to 90 degrees
- moved R4 4.18 mm to (180.8, 122.9)
- moved R5 4.18 mm to (182.9, 123.0)
- moved C2 3.07 mm to (202.6, 138.5)
- moved C5 3.07 mm to (202.6, 136.3)
- moved Y1 3.07 mm to (197.8, 137.4)
- moved J3 3.01 mm to (188.7, 97.6)
- moved C3 2.89 mm to (197.9, 133.0)
- moved C6 2.70 mm to (177.2, 124.7)
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Connections:
- net Net-(J1-PadA6) renamed DP
- net Net-(J1-PadA7) renamed DN
- REF** pad 12: ROW 2 -> (no net)
- REF** pad 31: (no net) -> ROW 2
- U1 pad 12: ROW 2 -> unconnected-(U1-Pad12)
- U1 pad 31: unconnected-(U1-Pad31) -> ROW 2
Routing:
- net +5V: track 18.6 -> 181.9 mm, vias 0 -> 5
- net GND: track 15.5 -> 131.5 mm, vias 0 -> 1
- net DP: track 0.00 -> 67.1 mm
- net DN: track 0.00 -> 65.7 mm
- net ROW 2: track 263.7 -> 320.6 mm, vias 2 -> 7
- net ROW3: track 301.1 -> 343.3 mm, vias 0 -> 2
- net RESET: track 3.06 -> 43.4 mm
- net ROW4: track 347.8 -> 375.8 mm
- net VCC: track 0.00 -> 27.3 mm, vias 0 -> 3
- net XTAL1: track 2.56 -> 16.8 mm
- net XTAL2: track 2.69 -> 15.1 mm
- net Net-(R6-Pad1): track 3.38 -> 12.3 mm
- net D-: track 2.94 -> 9.18 mm
- net D+: track 2.81 -> 9.05 mm
- net Net-(J1-PadA5): track 0.00 -> 5.83 mm
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