File: _autosave-Maja V1 PCB Redesign.kicad_pcb (KiCad board)
At the start: 2 copper layers, 345.1 x 138.7 mm, 166 parts, among them J1 TYPE-C-31-M-12, J2 AVR-ISP-6, K1 esc, K10 9, K11 0, K12 -, K13 =, K15 split backspace, K16 macro1, K17 tab, K18 q, K19 w, K2 1, K20 e, K21 r, K22 t, K23 y, K24 u, K25 i, K26 o, K27 p, K28 [, K29 ], K3 2, K30 \, K31 macro 2, K32 Caps, K33 a, K34 s, K35 d, K36 f, K37 g, K38 h, K39 j, K4 3, K40 k, K41 l, K42 ;, K43 ', K44 enter, K45 macro 3, K46 shift, K47 z, K48 x, K49 c, K5 4, K50 v, K51 b, K52 fn, K53 n, K54 m, K55 ,, K56 ., K57 /, K58 shift right, K59 up, K6 5, K60 ctrl left, K61 alt right, K62 space left, K63 code, K64 space right, K65 ctrl right, K66 left, K67 down, K68 right, K69 backspace, K7 6, K70 space left 2, K71 code 2, K72 Caps steped, K8 7, K9 8, U1 ATmega32U4-M, U2 PRTR5V0U2X, Y1 Crystal_GND24_Small

Commit message: add JST
Parts:
- moved R5 133.3 mm to (53.0, -100.6), turned to -90 degrees
- moved R4 115.8 mm to (51.0, -100.6), turned to -90 degrees
- moved U2 107.9 mm to (60.6, -132.6)
- moved F1 106.5 mm to (79.9, -141.2), turned to 0 degrees
- moved R2 97.6 mm to (88.5, -144.3), turned to 0 degrees
- moved R1 91.7 mm to (70.8, -144.3)
Changed lines of the file:
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@@
   )
   (footprint "Resistor_SMD:R_0805_2012Metric_Pad1.20x1.40mm_HandSolder" (layer "B.Cu")
-    (at 34.590176 -228.57095 180)
+    (at 70.768 -144.279 180)
     (descr "Resistor SMD 0805 (2012 Metric), square (rectangular) end terminal, IPC_7351 nominal with elongated pad for handsoldering. (Body size source: IPC-SM-782 page 72, https://www.pcb-3d.com/wordpress/wp-content/uploads/ipc-sm-782a_amendment_1_and_2.pdf), generated with kicad-footprint-generator")
     (tags "resistor handsolder")
@@
   )
   (footprint "random-keyboard-parts:SOT143B" (layer "B.Cu")
-    (at 24.950176 -234.38095 180)
+    (at 60.608 -132.595 180)
     (property "Sheetfile" "Maja V1 PCB Redesign.kicad_sch")
     (property "Sheetname" "")
@@
   )
   (footprint "Resistor_SMD:R_0805_2012Metric_Pad1.20x1.40mm_HandSolder" (layer "B.Cu")
-    (at 34.118926 -215.1622 180)
+    (at 50.956 -100.591 -90)
     (descr "Resistor SMD 0805 (2012 Metric), square (rectangular) end terminal, IPC_7351 nominal with elongated pad for handsoldering. (Body size source: IPC-SM-782 page 72, https://www.pcb-3d.com/wordpress/wp-content/uploads/ipc-sm-782a_amendment_1_and_2.pdf), generated with kicad-footprint-generator")
     (tags "resistor handsolder")
@@
     (property "Sheetname" "")
     (attr smd)
-    (fp_text reference "R4" (at 0 1.65) (layer "B.SilkS")
+    (fp_text reference "R4" (at 0 1.65 -270) (layer "B.SilkS")
       (effects (font (size 1 1) (thickness 0.15)) (justify mirror))
     )
-    (fp_text value "22" (at 0 -1.65) (layer "B.Fab")
+    (fp_text value "22" (at 0 -1.65 -270) (layer "B.Fab")
       (effects (font (size 1 1) (thickness 0.15)) (justify mirror))
     )
-    (fp_text user "${REFERENCE}" (at 0 0) (layer "B.Fab")
+    (fp_text user "${REFERENCE}" (at 0 0 -270) (layer "B.Fab")
       (effects (font (size 0.5 0.5) (thickness 0.08)) (justify mirror))
     )
@@
     (fp_line (start 1 0.625) (end 1 -0.625) (layer "B.Fab") (width 0.1))
     (fp_line (start -1 0.625) (end 1 0.625) (layer "B.Fab") (width 0.1))
-    (pad "1" smd roundrect (at -1 0 180) (size 1.2 1.4) (layers "B.Cu" "B.Paste" "B.Mask") (roundrect_rratio 0.208333)
+    (pad "1" smd roundrect (at -1 0 270) (size 1.2 1.4) (layers "B.Cu" "B.Paste" "B.Mask") (roundrect_rratio 0.208333)
       (net 65 "Net-(J1-PadA7)") (pintype "passive"))
-    (pad "2" smd roundrect (at 1 0 180) (size 1.2 1.4) (layers "B.Cu" "B.Paste" "B.Mask") (roundrect_rratio 0.208333)
+    (pad "2" smd roundrect (at 1 0 270) (size 1.2 1.4) (layers "B.Cu" "B.Paste" "B.Mask") (roundrect_rratio 0.208333)
       (net 89 "D-") (pintype "passive"))
     (model "${KICAD6_3DMODEL_DIR}/Resistor_SMD.3dshapes/R_0805_2012Metric.wrl"
@@
   )
   (footprint "Resistor_SMD:R_0805_2012Metric_Pad1.20x1.40mm_HandSolder" (layer "B.Cu")
-    (at 29.780176 -231.86095 180)
+    (at 52.988 -100.575 -90)
     (descr "Resistor SMD 0805 (2012 Metric), square (rectangular) end terminal, IPC_7351 nominal with elongated pad for handsoldering. (Body size source: IPC-SM-782 page 72, https://www.pcb-3d.com/wordpress/wp-content/uploads/ipc-sm-782a_amendment_1_and_2.pdf), generated with kicad-footprint-generator")
     (tags "resistor handsolder")
@@
     (property "Sheetname" "")
     (attr smd)
-    (fp_text reference "R5" (at 0 1.65) (layer "B.SilkS")
+    (fp_text reference "R5" (at 0 1.65 -270) (layer "B.SilkS")
       (effects (font (size 1 1) (thickness 0.15)) (justify mirror))
     )
-    (fp_text value "22" (at 0 -1.65) (layer "B.Fab")
+    (fp_text value "22" (at 0 -1.65 -270) (layer "B.Fab")
       (effects (font (size 1 1) (thickness 0.15)) (justify mirror))
     )
-    (fp_text user "${REFERENCE}" (at 0 0) (layer "B.Fab")
+    (fp_text user "${REFERENCE}" (at 8.62 1.016 -270) (layer "B.Fab")
       (effects (font (size 0.5 0.5) (thickness 0.08)) (justify mirror))
     )
@@
     (fp_line (start -1 -0.625) (end -1 0.625) (layer "B.Fab") (width 0.1))
     (fp_line (start 1 0.625) (end 1 -0.625) (layer "B.Fab") (width 0.1))
-    (pad "1" smd roundrect (at -1 0 180) (size 1.2 1.4) (layers "B.Cu" "B.Paste" "B.Mask") (roundrect_rratio 0.208333)
+    (pad "1" smd roundrect (at -1 0 270) (size 1.2 1.4) (layers "B.Cu" "B.Paste" "B.Mask") (roundrect_rratio 0.208333)
       (net 66 "Net-(J1-PadA6)") (pintype "passive"))
-    (pad "2" smd roundrect (at 1 0 180) (size 1.2 1.4) (layers "B.Cu" "B.Paste" "B.Mask") (roundrect_rratio 0.208333)
+    (pad "2" smd roundrect (at 1 0 270) (size 1.2 1.4) (layers "B.Cu" "B.Paste" "B.Mask") (roundrect_rratio 0.208333)
       (net 90 "D+") (pintype "passive"))
     (model "${KICAD6_3DMODEL_DIR}/Resistor_SMD.3dshapes/R_0805_2012Metric.wrl"
@@
   )
   (footprint "Resistor_SMD:R_0805_2012Metric_Pad1.20x1.40mm_HandSolder" (layer "B.Cu")
-    (at 34.590176 -225.62095 180)
+    (at 88.548 -144.279)
     (descr "Resistor SMD 0805 (2012 Metric), square (rectangular) end terminal, IPC_7351 nominal with elongated pad for handsoldering. (Body size source: IPC-SM-782 page 72, https://www.pcb-3d.com/wordpress/wp-content/uploads/ipc-sm-782a_amendment_1_and_2.pdf), generated with kicad-footprint-generator")
     (tags "resistor handsolder")
@@
     (fp_line (start 1 -0.625) (end -1 -0.625) (layer "B.Fab") (width 0.1))
     (fp_line (start 1 0.625) (end 1 -0.625) (layer "B.Fab") (width 0.1))
-    (pad "1" smd roundrect (at -1 0 180) (size 1.2 1.4) (layers "B.Cu" "B.Paste" "B.Mask") (roundrect_rratio 0.208333)
+    (pad "1" smd roundrect (at -1 0) (size 1.2 1.4) (layers "B.Cu" "B.Paste" "B.Mask") (roundrect_rratio 0.208333)
       (net 68 "Net-(J1-PadA5)") (pintype "passive"))
-    (pad "2" smd roundrect (at 1 0 180) (size 1.2 1.4) (layers "B.Cu" "B.Paste" "B.Mask") (roundrect_rratio 0.208333)
+    (pad "2" smd roundrect (at 1 0) (size 1.2 1.4) (layers "B.Cu" "B.Paste" "B.Mask") (roundrect_rratio 0.208333)
       (net 2 "GND") (pintype "passive"))
     (model "${KICAD6_3DMODEL_DIR}/Resistor_SMD.3dshapes/R_0805_2012Metric.wrl"
@@
   )
   (footprint "Fuse:Fuse_1206_3216Metric_Pad1.42x1.75mm_HandSolder" (layer "B.Cu")
-    (at 34.760176 -237.71095 180)
+    (at 79.9485 -141.231)
     (descr "Fuse SMD 1206 (3216 Metric), square (rectangular) end terminal, IPC_7351 nominal with elongated pad for handsoldering. (Body size source: http://www.tortai-tech.com/upload/download/2011102023233369053.pdf), generated with kicad-footprint-generator")
     (tags "fuse handsolder")
@@
     (fp_line (start 1.6 0.8) (end 1.6 -0.8) (layer "B.Fab") (width 0.1))
     (fp_line (start -1.6 -0.8) (end -1.6 0.8) (layer "B.Fab") (width 0.1))
-    (pad "1" smd roundrect (at -1.4875 0 180) (size 1.425 1.75) (layers "B.Cu" "B.Paste" "B.Mask") (roundrect_rratio 0.175439)
+    (pad "1" smd roundrect (at -1.4875 0) (size 1.425 1.75) (layers "B.Cu" "B.Paste" "B.Mask") (roundrect_rratio 0.175439)
       (net 4 "+5V") (pintype "passive"))
-    (pad "2" smd roundrect (at 1.4875 0 180) (size 1.425 1.75) (layers "B.Cu" "B.Paste" "B.Mask") (roundrect_rratio 0.175439)
+    (pad "2" smd roundrect (at 1.4875 0) (size 1.425 1.75) (layers "B.Cu" "B.Paste" "B.Mask") (roundrect_rratio 0.175439)
       (net 64 "VCC") (pintype "passive"))
     (model "${KICAD6_3DMODEL_DIR}/Fuse.3dshapes/Fuse_1206_3216Metric.wrl"
