File: Matrix.kicad_sch (KiCad schematic)
At the start: 140 parts, among them K1 esc, K10 9, K11 0, K12 -, K13 =, K15 split backspace, K16 macro1, K17 tab, K18 q, K19 w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

Commit message: LCSC Component
Parts:
- D1, D10, D11, D12, D13, D14, D15, D16, D17, D18, D19, D2, D20, D21, D22, D23, D24, D25, D26, D27, D28, D29, D3, D30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: LCSC (none) -> C77978
